File: FSR_matrix_readout/FSR_matrix_readout.kicad_sch (KiCad schematic)
At the start: 7 parts, among them U1 NCD98010XMXTAG, U17 74VHC393FT, U2 NCD98010XMXTAG, U3 TLV9064, U4 TPW4051-QF4R, U5 TPW4051-QF4R

Commit message: done sense opamp module
Parts:
- removed R1: 330R, symbol Device:R_US
- removed U3: TLV9064, symbol Amplifier_Operational:TLV9064
- added FPC1, FPC2: AFA07-S16FCC-00, easyeda2kicad:FPC-SMD_16P-P1.00_AFA07-S16FCC-00, symbol lcsc:AFA07-S16FCC-00
Connections:
- new net fsr_drive0: FPC1.1
- new net fsr_drive1: FPC1.2
- new net fsr_drive10: FPC1.11
- new net fsr_drive11: FPC1.12
- new net fsr_drive12: FPC1.13
- new net fsr_drive13: FPC1.14
- new net fsr_drive14: FPC1.15
- new net fsr_drive15: FPC1.16
- new net fsr_drive2: FPC1.3
- new net fsr_drive3: FPC1.4
- new net fsr_drive4: FPC1.5
- new net fsr_drive5: FPC1.6
- new net fsr_drive6: FPC1.7
- new net fsr_drive7: FPC1.8
- new net fsr_drive8: FPC1.9
- new net fsr_drive9: FPC1.10
- new net fsr_i_out0: FPC2.1
- new net fsr_i_out1: FPC2.2
- new net fsr_i_out10: FPC2.11
- new net fsr_i_out11: FPC2.12
- new net fsr_i_out12: FPC2.13
- new net fsr_i_out13: FPC2.14
- new net fsr_i_out14: FPC2.15
- new net fsr_i_out15: FPC2.16
- new net fsr_i_out2: FPC2.3
- new net fsr_i_out3: FPC2.4
- new net fsr_i_out4: FPC2.5
- new net fsr_i_out5: FPC2.6
- new net fsr_i_out6: FPC2.7
- new net fsr_i_out7: FPC2.8
- new net fsr_i_out8: FPC2.9
- new net fsr_i_out9: FPC2.10
- no-connect marks 0 -> 4
Other:
- added sheet sense_opamps (sense_opamps.kicad_sch)
- sheet frontend_mux ports: added V_{g}, fsr_drive[0..15], sel[0..15]; removed none
- note removed: "R_{f} for opamp"
- moved on the sheet: U1, U17, U2

Commit message: add addr_counter
Parts:
- removed U17: 74VHC393FT, easyeda2kicad:TSSOP-14_L5.0-W4.4-P0.65-LS6.4-BL, symbol lcsc:74VHC393FT
Other:
- added sheet addr_counter (addr_counter.kicad_sch)
- moved on the sheet: U1, U2
Changed lines of the file:
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@@
-	)
-	(symbol
-		(lib_id "lcsc:74VHC393FT")
-		(at 135.89 102.87 0)
-		(unit 1)
-		(body_style 1)
-		(exclude_from_sim no)
-		(in_bom yes)
-		(on_board yes)
-		(in_pos_files yes)
-		(dnp no)
-		(fields_autoplaced yes)
-		(property "Reference" "U17"
-			(at 135.89 87.63 0)
-			(show_name no)
-			(do_not_autoplace no)
-			(effects
-				(font
-					(size 1.27 1.27)
-				)
-			)
-		)
-		(property "Value" "74VHC393FT"
-			(at 135.89 90.17 0)
-			(show_name no)
-			(do_not_autoplace no)
-			(effects
-				(font
-					(size 1.27 1.27)
-				)
-			)
-		)
-		(property "Footprint" "easyeda2kicad:TSSOP-14_L5.0-W4.4-P0.65-LS6.4-BL"
-			(at 135.89 118.11 0)
-			(hide yes)
-			(show_name no)
-			(do_not_autoplace no)
-			(effects
-				(font
-					(size 1.27 1.27)
-				)
-			)
-		)
-		(property "Datasheet" "https://www.lcsc.com/datasheet/C5331508.pdf"
-			(at 135.89 120.65 0)
-			(hide yes)
-			(show_name no)
-			(do_not_autoplace no)
-			(effects
-				(font
-					(size 1.27 1.27)
-				)
-			)
-		)
-		(property "Description" ""
-			(at 135.89 102.87 0)
-			(hide yes)
-			(show_name no)
-			(do_not_autoplace no)
-			(effects
-				(font
-					(size 1.27 1.27)
-				)
-			)
-		)
-		(property "Manufacturer" "TOSHIBA(东芝)"
-			(at 135.89 123.19 0)
-			(hide yes)
-			(show_name no)
-			(do_not_autoplace no)
-			(effects
-				(font
-					(size 1.27 1.27)
-				)
-			)
-		)
-		(property "MPN" "74VHC393FT(BJ)"
-			(at 135.89 125.73 0)
-			(hide yes)
-			(show_name no)
-			(do_not_autoplace no)
-			(effects
-				(font
-					(size 1.27 1.27)
-				)
-			)
-		)
-		(property "LCSC Part" "C5331508"
-			(at 135.89 128.27 0)
-			(hide yes)
-			(show_name no)
-			(do_not_autoplace no)
-			(effects
-				(font
-					(size 1.27 1.27)
-				)
-			)
-		)
-		(pin "5"
-		)
-		(pin "10"
-		)
-		(pin "12"
-		)
-		(pin "14"
-		)
-		(pin "4"
-		)
-		(pin "2"
-		)
-		(pin "1"
-		)
-		(pin "3"
-		)
-		(pin "7"
-		)
-		(pin "8"
-		)
-		(pin "6"
-		)
-		(pin "9"
-		)
-		(pin "11"
-		)
-		(pin "13"
-		)
-		(instances
-			(project "FSR_matrix_readout"
-				(path "/6dca5e5c-f676-465d-98c9-14af6047a226"
-					(reference "U17")
-					(unit 1)
-				)
-			)
-		)
 	)
 	(symbol
 		(lib_id "lcsc:NCD98010XMXTAG")
-		(at 124.46 66.04 0)
+		(at 220.98 66.04 0)
 		(unit 1)
 		(body_style 1)
@@
 		(fields_autoplaced yes)
 		(property "Reference" "U2"
-			(at 124.46 54.61 0)
+			(at 220.98 54.61 0)
 			(show_name no)
 			(do_not_autoplace no)
@@
 		)
 		(property "Value" "NCD98010XMXTAG"
-			(at 124.46 57.15 0)
+			(at 220.98 57.15 0)
 			(show_name no)
 			(do_not_autoplace no)
@@
 		)
 		(property "Footprint" "easyeda2kicad:X2QFN-8_L1.5-W1.5-P0.50-BL"
-			(at 124.46 77.47 0)
+			(at 220.98 77.47 0)
 			(hide yes)
 			(show_name no)
@@
 		)
 		(property "Datasheet" "https://www.lcsc.com/datasheet/C895632.pdf"
-			(at 124.46 80.01 0)
+			(at 220.98 80.01 0)
 			(hide yes)
 			(show_name no)
@@
 		)
 		(property "Description" ""
-			(at 124.46 66.04 0)
+			(at 220.98 66.04 0)
 			(hide yes)
 			(show_name no)
@@
 		)
 		(property "Manufacturer" "onsemi(安森美)"
-			(at 124.46 82.55 0)
+			(at 220.98 82.55 0)
 			(hide yes)
 			(show_name no)
@@
 		)
 		(property "MPN" "NCD98010XMXTAG"
-			(at 124.46 85.09 0)
+			(at 220.98 85.09 0)
 			(hide yes)
 			(show_name no)
@@
 		)
 		(property "LCSC Part" "C895632"
-			(at 124.46 87.63 0)
+			(at 220.98 87.63 0)
 			(hide yes)
 			(show_name no)
@@
 	(symbol
 		(lib_id "lcsc:NCD98010XMXTAG")
-		(at 124.46 44.45 0)
+		(at 220.98 44.45 0)
 		(unit 1)
 		(body_style 1)
@@
 		(fields_autoplaced yes)
 		(property "Reference" "U1"
-			(at 124.46 33.02 0)
+			(at 220.98 33.02 0)
 			(show_name no)
 			(do_not_autoplace no)
@@
 		)
 		(property "Value" "NCD98010XMXTAG"
-			(at 124.46 35.56 0)
+			(at 220.98 35.56 0)
 			(show_name no)
 			(do_not_autoplace no)
@@
 		)
 		(property "Footprint" "easyeda2kicad:X2QFN-8_L1.5-W1.5-P0.50-BL"
-			(at 124.46 55.88 0)
+			(at 220.98 55.88 0)
 			(hide yes)
 			(show_name no)
@@
 		)
 		(property "Datasheet" "https://www.lcsc.com/datasheet/C895632.pdf"
-			(at 124.46 58.42 0)
+			(at 220.98 58.42 0)
 			(hide yes)
 			(show_name no)
@@
 		)
 		(property "Description" ""
-			(at 124.46 44.45 0)
+			(at 220.98 44.45 0)
 			(hide yes)
 			(show_name no)
@@
 		)
 		(property "Manufacturer" "onsemi(安森美)"
-			(at 124.46 60.96 0)
+			(at 220.98 60.96 0)
 			(hide yes)
 			(show_name no)
@@
 		)
 		(property "MPN" "NCD98010XMXTAG"
-			(at 124.46 63.5 0)
+			(at 220.98 63.5 0)
 			(hide yes)
 			(show_name no)
@@
 		)
 		(property "LCSC Part" "C895632"
-			(at 124.46 66.04 0)
+			(at 220.98 66.04 0)
 			(hide yes)
 			(show_name no)
@@
 	)
 	(sheet
-		(at 158.75 43.18)
+		(at 157.48 36.83)
 		(size 22.86 7.62)
 		(exclude_from_sim no)
@@
 		)
 		(property "Sheetname" "16:1_decoder"
-			(at 158.75 42.4684 0)
+			(at 157.48 36.1184 0)
 			(show_name no)
 			(do_not_autoplace no)
@@
 		)
 		(property "Sheetfile" "16_to_1_decoder.kicad_sch"
-			(at 158.75 51.3846 0)
+			(at 157.48 45.0346 0)
 			(show_name no)
 			(do_not_autoplace no)
@@
 		)
 		(pin "a[0..3]" input
-			(at 158.75 46.99 180)
+			(at 157.48 40.64 180)
 			(effects
 				(font
@@
 		)
 		(pin "d[0..15]" output
-			(at 181.61 46.99 0)
+			(at 180.34 40.64 0)
 			(effects
 				(font
@@
 				)
 			)
+		)
+	)
+	(sheet
+		(at 115.57 35.56)
+		(size 26.67 8.89)
+		(exclude_from_sim no)
+		(in_bom yes)
+		(on_board yes)
+		(dnp no)
+		(fields_autoplaced yes)
+		(stroke
+			(width 0.1524)
+			(type solid)
+		)
+		(fill
+			(color 0 0 0 0)
+		)
+		(property "Sheetname" "addr_counter"
+			(at 115.57 34.8484 0)
+			(show_name no)
+			(do_not_autoplace no)
+			(effects
+				(font
+					(size 1.27 1.27)
+				)
+				(justify left bottom)
+			)
+		)
+		(property "Sheetfile" "addr_counter.kicad_sch"
+			(at 115.57 45.0346 0)
+			(show_name no)
+			(do_not_autoplace no)
+			(effects
+				(font
+					(size 1.27 1.27)
+				)
+				(justify left top)
+			)
+		)
+		(property "Field2" ""
+			(at 115.57 35.56 0)
+			(hide yes)
+			(show_name no)
+			(do_not_autoplace no)
+			(effects
+				(font
+					(size 1.27 1.27)
+				)
+			)
+		)
+		(pin "drive_a[0..3]" output
+			(at 142.24 38.1 0)
+			(effects
+				(font
+					(size 1.27 1.27)
+				)
+				(justify right)
+			)
+		)
+		(pin "~{clk}" input
+			(at 115.57 38.1 180)
+			(effects
+				(font
+					(size 1.27 1.27)
+				)
+				(justify left)
+			)
+		)
+		(pin "sense_a[0..2]" output
+			(at 142.24 40.64 0)
+			(effects
+				(font
+					(size 1.27 1.27)
+				)
+				(justify right)
+			)
+		)
+		(pin "clr" input
+			(at 115.57 40.64 180)
+			(effects
+				(font
+					(size 1.27 1.27)
+				)
+				(justify left)
+			)
+		)
+		(instances
+			(project "FSR_matrix_readout"
+				(path "/6dca5e5c-f676-465d-98c9-14af6047a226"
+					(page "5")
+				)
+			)
