File: internal_adc_pcb/fsr_matrix_readout_internal_adc.kicad_pcb (KiCad board)
At the start: 2 copper layers, 50 x 65 mm, 97 parts, among them J1 Conn_01x22, J2 Conn_01x22, U1 RS2323XUTQK10, U10 TLV9061xDBV, U11 SN74AHC138RGYR, U12 SN74AHC138RGYR, U13 SN74LVC1G14DCKR_C19829630, U14 TLV9064, U15 TLV9064, U16 TLV9064, U17 TLV9064, U2 RS2323XUTQK10, U3 RS2323XUTQK10, U4 RS2323XUTQK10, U5 RS2323XUTQK10, U6 RS2323XUTQK10, U7 RS2323XUTQK10, U8 RS2323XUTQK10, U9 TPS7A2033PDBVR

Commit message: adjust for production
Parts:
- renumbered TP_VG to TP_VG1, TP_VG to TP_VG2
